File: 901p-board-v2/901p-board-v2.kicad_sch (KiCad schematic)
At the start: 32 parts, among them J1 USB-C (USB2.0, 14-pin), J2 DE15, J3 MICRO USB-B, Q1 PMOS, SW1 SW_Push, U1 HUSB238_xxxDD, U2 TPS82140, U3 ESP32-S3-WROOM-1, U4 MAX3232, U5 NHD-C0220BIZ

Commit message: v2 board stuff
Parts:
- removed C2: 10µF, symbol Device:C
- removed C3: 430pF, symbol Device:C
- removed C4: 22µF, symbol Device:C
- removed D1, D2: B340AXF, symbol Device:D_Schottky
- removed J3: MICRO USB-B, symbol Connector:USB_B_Micro
- removed R5: 309kΩ, symbol Device:R
- removed R6: 100kΩ, symbol Device:R
- removed R7: 5.1k, symbol Device:R
- removed SW1: SW_Push, symbol Switch:SW_Push
- removed TP1: AO+, symbol Connector:TestPoint
- removed TP2: AO-, symbol Connector:TestPoint
- removed U2: TPS82140, Package_LGA:Texas_SIL0008D_MicroSiP-8-1EP_2.8x3mm_P0.65mm_EP1.1x1.9mm_ThermalVias, symbol Converter_DCDC:TPS82140
- removed U3: ESP32-S3-WROOM-1, RF_Module:ESP32-S3-WROOM-1, symbol RF_Module:ESP32-S3-WROOM-1
- added C10: 10µF, Capacitor_SMD:C_0805_2012Metric_Pad1.18x1.45mm_HandSolder, symbol Device:C
- added C12: 100nF, Capacitor_SMD:C_0805_2012Metric_Pad1.18x1.45mm_HandSolder, symbol Device:C
- added C13, C14, C15: 22µF, Capacitor_SMD:C_0805_2012Metric_Pad1.18x1.45mm_HandSolder, symbol Device:C
- added C6: 100nF, Capacitor_SMD:C_0805_2012Metric_Pad1.18x1.45mm_HandSolder, symbol Device:C_Small
- added C7: 10pF, Capacitor_SMD:C_0805_2012Metric_Pad1.18x1.45mm_HandSolder, symbol Device:C_Small
- added J3: AO(+/-), Connector_PinHeader_1.00mm:PinHeader_1x02_P1.00mm_Vertical, symbol Connector:Conn_01x02_Pin
- added L1: 1 μH, Inductor_SMD:L_1210_3225Metric_Pad1.42x2.65mm_HandSolder, symbol Device:L
- added R5, R6: 1MΩ, Resistor_SMD:R_0805_2012Metric_Pad1.20x1.40mm_HandSolder, symbol Device:R_US
- added R7: 110kΩ, Resistor_SMD:R_0805_2012Metric_Pad1.20x1.40mm_HandSolder, symbol Device:R_US
- added U3: ESP32-S3-DevKitC, PCM_Espressif:ESP32-S3-DevKitC, symbol PCM_Espressif:ESP32-S3-DevKitC
- added U6: TPS63060, Package_SON:Texas_S-PWSON-N10_ThermalVias, symbol Regulator_Switching:TPS63060
- C1, C9: footprint (none) -> Capacitor_SMD:C_0805_2012Metric_Pad1.18x1.45mm_HandSolder
- C11: value 1µF -> 10µF; footprint (none) -> Capacitor_SMD:C_0805_2012Metric_Pad1.18x1.45mm_HandSolder
- C2: renamed from C5; footprint (none) -> Capacitor_SMD:C_0805_2012Metric_Pad1.18x1.45mm_HandSolder
- C3: renamed from C6; footprint (none) -> Capacitor_SMD:C_0805_2012Metric_Pad1.18x1.45mm_HandSolder
- C4: renamed from C8; footprint (none) -> Capacitor_SMD:C_0805_2012Metric_Pad1.18x1.45mm_HandSolder
- C5: renamed from C7; footprint (none) -> Capacitor_SMD:C_0805_2012Metric_Pad1.18x1.45mm_HandSolder
- C8: renamed from C10; footprint (none) -> Capacitor_SMD:C_0805_2012Metric_Pad1.18x1.45mm_HandSolder
- J1: value USB-C (USB2.0, 14-pin) -> USB-C (14 pins); footprint (none) -> footprints:UJ20-C-H-G-SMT-2A-P16-TR
- J2: footprint (none) -> footprints:AMPHENOL_10090926-P154XLF
- Q1: footprint (none) -> footprints:PPAK3x3
- R1, R2, R3, R4: footprint (none) -> Resistor_SMD:R_0805_2012Metric_Pad1.20x1.40mm_HandSolder
- U4: footprint (none) -> Package_SO:SOIC-16W_5.3x10.2mm_P1.27mm
Connections:
- net +3.3V: now also C12.1, U3.1 (3V3), U3.2 (3V3)
- net AO+: now also J3.1 (Pin_1)
- net AO-: now also J3.2 (Pin_2)
- net GND: now also C11.2, C10.2, C12.2, C13.2, C14.2, C15.2, C6.2, C7.2, R7.2, U3.22 (GND), U3.23 (GND), U3.24 (GND), U3.44 (GND), U6.11 (PGND), U6.4 (PS/SYNC), U6.7 (GND); no longer C11.1
- net VBUS: now also C11.1, C10.1, U6.2 (VIN), U6.3 (EN)
- new net: C7.1, R6.2, R7.1, U6.8 (FB)
- new net: L1.1, U6.1 (L1)
- new net: L1.2, U6.10 (L2)
- new net: R5.2, U6.5 (PG)
- new net: C6.1, U6.6 (VAUX)
- new net +5V: C13.1, C14.1, C15.1, R5.1, R6.1, U3.21 (5V), U6.9 (VOUT)
- no-connect marks 6 -> 50
Other:
- moved on the sheet: C8, C9, U5

Commit message: finish v2 board
Parts:
- added C16: 100nF, Capacitor_SMD:C_0805_2012Metric_Pad1.18x1.45mm_HandSolder, symbol Device:C
- added R8, R9: 5.1kΩ, Resistor_SMD:R_0805_2012Metric_Pad1.20x1.40mm_HandSolder, symbol Device:R
- J3: footprint Connector_PinHeader_1.00mm:PinHeader_1x02_P1.00mm_Vertical -> Connector_PinHeader_2.54mm:PinHeader_1x02_P2.54mm_Vertical
Connections:
- net +3.3V: now also C16.1; no longer C8.1
- net GND: now also C8.2, C16.2, R8.2, R9.2
- net SCL: now also U3.32 (GPIO35), R9.1
- net SDA: now also U3.33 (GPIO36), R8.1
- net SER_RX: now also U3.37 (GPIO40/MTDO)
- net SER_TX: now also U3.36 (GPIO39/MTCK)
- net VBUS: now also Q1.1 (D); no longer Q1.3 (S)
- net at J1.A4 (VBUS), J1.A9 (VBUS), J1.B4 (VBUS)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: now also Q1.3 (S); no longer Q1.1 (D)
- net at U5.6 (VOUT): now also C8.1; no longer C8.2
- no-connect marks 50 -> 46
Other:
- moved on the sheet: C8, C9, U3, U5

Commit message: final review i think
Connections:
- net +3.3V: now also R8.1, R9.1
- net GND: now also U4.10 (T2IN), U4.8 (R2IN); no longer R8.2, R9.2
- net SCL: now also R9.2; no longer R9.1
- net SDA: now also R8.2; no longer R8.1
- no-connect marks 46 -> 44
Other:
- moved on the sheet: R8, R9
