File: 901p-board-v2/901p-board-v2.kicad_sch (KiCad schematic)
At the start: 35 parts, among them J1 USB-C (14 pins), J2 DE15, J3 AO(+/-), Q1 PMOS, U1 HUSB238_xxxDD, U3 ESP32-S3-DevKitC, U4 MAX3232, U5 NHD-C0220BIZ, U6 TPS63060

Commit message: cleanup stuff
Parts:
- C1, C8, C9: Digikey (none) -> 1276-6470-1-ND
- C10, C11: Digikey (none) -> 1276-6457-1-ND
- C12, C16, C2, C3, C4, C5, C6: Digikey (none) -> 1276-1003-1-ND
- C13, C14, C15: Digikey (none) -> 1276-6501-1-ND
- C7: Digikey (none) -> 1276-2561-1-ND
- J1: Digikey (none) -> 2223-UJ20-C-H-G-SMT-2A-P16-TRCT-ND
- J2: Digikey (none) -> 10090926-P154XLF
- J3, U1, U3: now left out of the parts list
- L1: Digikey (none) -> 490-18403-1-ND
- Q1: value PMOS -> AONR21357; Digikey (none) -> 785-AONR21357CT-ND
- R1: Digikey (none) -> 311-10.0CRCT-ND
- R2: Digikey (none) -> 311-10.0KCRCT-ND
- R3, R8, R9: Digikey (none) -> 311-5.1KARCT-ND
- R4: Digikey (none) -> 311-49.9KCRCT-ND
- R5, R6: Digikey (none) -> 311-1.00MCRCT-ND
- R7: Digikey (none) -> 311-110KARCT-ND
- U4: value MAX3232 -> MAX3232CDR; footprint Package_SO:SOIC-16W_5.3x10.2mm_P1.27mm -> footprints:D16; Digikey (none) -> 296-13094-1-ND
- U5: Digikey (none) -> NHD-C0220BIZ-FSW-FBW-3V3M-ND
- U6: value TPS63060 -> TPS63060DSCR; Digikey (none) -> 296-30204-1-ND
Other:
- moved on the sheet: C10, C11, C13, C14, C15, C16, C6, C7, C8, C9, L1, R5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
