File: 901p-board-v2/901p-board-v2.kicad_pcb (KiCad board)
At the start: 2 copper layers, 104.7 x 74.6 mm, 36 parts, among them J1 USB-C (14 pins), J2 DE15, J3 AO(+/-), Q1 PMOS, U1 HUSB238_xxxDD, U3 ESP32-S3-DevKitC, U4 MAX3232, U5 NHD-C0220BIZ, U6 TPS63060

Commit message: cleanup stuff
Parts:
- Q1: value PMOS -> AONR21357
- U4: value MAX3232 -> MAX3232CDW; footprint Package_SO:SOIC-16W_5.3x10.2mm_P1.27mm -> footprints:D16
- U6: value TPS63060 -> TPS63060DSCT
- moved C2 1.73 mm to (106.6, 114.4)
- moved C3 1.73 mm to (103.6, 115.6)
- moved C4 1.73 mm to (107.7, 116.5)
- moved C5 1.70 mm to (100.8, 115.5)
- moved U4 0.74 mm to (103.2, 121.4)
Routing:
- net /SCL: track 74.1 -> 77.5 mm
- net Net-(J1-CC1): track 3.31 -> 4.50 mm
- net /SDA: track 74.0 -> 75.0 mm
- net GND: track 8.61 -> 7.89 mm, vias 15 -> 194
